File: eagle/project_l432/linetracer/linetracer.brd (EAGLE design)
At the start: 160 x 100 mm, 2 parts

Commit message: power
Parts:
- added C1: 0.1μ, rcl:C025-024X044
- added C2: 47μ, rcl:E5-10,5
- added IC1: TA4805S, TA4805S:TO230P250X680X1080-3P
- added LED1: (no value), led:LED3MM
- added Q1: IRFU5505PBF, IRFU5505PBF:TO229P239X654X978-3P
- added R1, R3: 100k, rcl:0204V
- added R2: 4.7k, rcl:0204V
- added R4: 22k, rcl:0204V
- added U$2: TOGGLE-SWITCH, toggle-switch:1X03
Connections:
- new net +5V: C2.+, IC1.3
- new net BATTERY: R3.1, R4.2
- new net GND: C1.2, C2.-, IC1.2, JP1.1, LED1.K, R4.1, U$2.1
- new net N$1: JP1.2, Q1.3, R1.2
- new net N$2: Q1.1, R1.1, U$2.2
- new net N$4: C1.1, IC1.1, Q1.2, R2.2, R3.2
- new net N$5: LED1.A, R2.1
Changed lines of the file:
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@@
 </element>
 <element name="U$1" library="nucleo32.Ibr" package="NUCLEO_L432KC" value="NUCLEO_L432KC" x="49.53" y="64.77" smashed="yes"/>
+<element name="IC1" library="TA4805S" package="TO230P250X680X1080-3P" value="TA4805S" x="24.13" y="45.72" smashed="yes" rot="R180">
+<attribute name="DESCRIPTION" value="Bipolar linear IC" x="24.13" y="45.72" size="1.778" layer="27" rot="R180" display="off"/>
+<attribute name="HEIGHT" value="2.5mm" x="24.13" y="45.72" size="1.778" layer="27" rot="R180" display="off"/>
+<attribute name="MANUFACTURER_NAME" value="Toshiba" x="24.13" y="45.72" size="1.778" layer="27" rot="R180" display="off"/>
+<attribute name="MANUFACTURER_PART_NUMBER" value="TA4805F" x="24.13" y="45.72" size="1.778" layer="27" rot="R180" display="off"/>
+<attribute name="MOUSER_PART_NUMBER" value="" x="24.13" y="45.72" size="1.778" layer="27" rot="R180" display="off"/>
+<attribute name="MOUSER_PRICE-STOCK" value="" x="24.13" y="45.72" size="1.778" layer="27" rot="R180" display="off"/>
+<attribute name="NAME" x="24.13" y="46.99" size="1.27" layer="25" rot="R180" align="center"/>
+<attribute name="RS_PART_NUMBER" value="" x="24.13" y="45.72" size="1.778" layer="27" rot="R180" display="off"/>
+<attribute name="RS_PRICE-STOCK" value="" x="24.13" y="45.72" size="1.778" layer="27" rot="R180" display="off"/>
+<attribute name="VALUE" x="22.86" y="44.45" size="1.27" layer="27" rot="R180" align="center"/>
+</element>
+<element name="Q1" library="IRFU5505PBF" package="TO229P239X654X978-3P" value="IRFU5505PBF" x="5.08" y="-6.35" smashed="yes">
+<attribute name="ALLIED_NUMBER" value="70017047" x="5.08" y="-6.35" size="1.778" layer="27" display="off"/>
+<attribute name="ALLIED_PRICE-STOCK" value="https://www.alliedelec.com/infineon-irfu5505pbf/70017047/" x="5.08" y="-6.35" size="1.778" layer="27" display="off"/>
+<attribute name="DESCRIPTION" value="INFINEON - IRFU5505PBF - MOSFET, P, -55V, -18A, I-PAK" x="5.08" y="-6.35" size="1.778" layer="27" display="off"/>
+<attribute name="HEIGHT" value="2.39mm" x="5.08" y="-6.35" size="1.778" layer="27" display="off"/>
+<attribute name="MANUFACTURER_NAME" value="Infineon" x="5.08" y="-6.35" size="1.778" layer="27" display="off"/>
+<attribute name="MANUFACTURER_PART_NUMBER" value="IRFU5505PBF" x="5.08" y="-6.35" size="1.778" layer="27" display="off"/>
+<attribute name="MOUSER_PART_NUMBER" value="942-IRFU5505PBF" x="5.08" y="-6.35" size="1.778" layer="27" display="off"/>
+<attribute name="MOUSER_PRICE-STOCK" value="https://www.mouser.com/Search/Refine.aspx?Keyword=942-IRFU5505PBF" x="5.08" y="-6.35" size="1.778" layer="27" display="off"/>
+<attribute name="NAME" x="5.08" y="-6.35" size="1.27" layer="25" align="center"/>
+<attribute name="RS_PART_NUMBER" value="" x="5.08" y="-6.35" size="1.778" layer="27" display="off"/>
+<attribute name="RS_PRICE-STOCK" value="" x="5.08" y="-6.35" size="1.778" layer="27" display="off"/>
+<attribute name="VALUE" x="5.08" y="-6.35" size="1.27" layer="27" align="center"/>
+</element>
+<element name="U$2" library="toggle-switch" package="1X03" value="TOGGLE-SWITCH" x="15.24" y="34.29" smashed="yes">
+<attribute name="NAME" x="11.3538" y="36.1188" size="1.27" layer="25" ratio="10"/>
+<attribute name="VALUE" x="11.43" y="31.115" size="1.27" layer="27"/>
+</element>
+<element name="R1" library="rcl" library_urn="urn:adsk.eagle:library:334" package="0204V" package3d_urn="urn:adsk.eagle:package:23495/1" value="100k" x="13.97" y="26.67" smashed="yes">
+<attribute name="NAME" x="11.8364" y="27.8384" size="1.27" layer="25" ratio="10"/>
+<attribute name="SPICEPREFIX" value="R" x="13.97" y="26.67" size="1.778" layer="27" display="off"/>
+<attribute name="VALUE" x="11.8364" y="24.3586" size="1.27" layer="27" ratio="10"/>
+</element>
+<element name="R2" library="rcl" library_urn="urn:adsk.eagle:library:334" package="0204V" package3d_urn="urn:adsk.eagle:package:23495/1" value="4.7k" x="2.54" y="-11.43" smashed="yes">
+<attribute name="NAME" x="0.4064" y="-10.2616" size="1.27" layer="25" ratio="10"/>
+<attribute name="SPICEPREFIX" value="R" x="2.54" y="-11.43" size="1.778" layer="27" display="off"/>
+<attribute name="VALUE" x="0.4064" y="-13.7414" size="1.27" layer="27" ratio="10"/>
+</element>
+<element name="LED1" library="led" library_urn="urn:adsk.eagle:library:259" package="LED3MM" package3d_urn="urn:adsk.eagle:package:15797/1" value="" x="12.7" y="15.24" smashed="yes">
+<attribute name="NAME" x="14.605" y="15.621" size="1.27" layer="25" ratio="10"/>
+<attribute name="VALUE" x="14.605" y="13.589" size="1.27" layer="27" ratio="10"/>
+</element>
+<element name="R3" library="rcl" library_urn="urn:adsk.eagle:library:334" package="0204V" package3d_urn="urn:adsk.eagle:package:23495/1" value="100k" x="2.54" y="-17.78" smashed="yes">
+<attribute name="NAME" x="0.4064" y="-16.6116" size="1.27" layer="25" ratio="10"/>
+<attribute name="SPICEPREFIX" value="R" x="2.54" y="-17.78" size="1.778" layer="27" display="off"/>
+<attribute name="VALUE" x="0.4064" y="-20.0914" size="1.27" layer="27" ratio="10"/>
+</element>
+<element name="R4" library="rcl" library_urn="urn:adsk.eagle:library:334" package="0204V" package3d_urn="urn:adsk.eagle:package:23495/1" value="22k" x="2.54" y="-24.13" smashed="yes">
+<attribute name="NAME" x="0.4064" y="-22.9616" size="1.27" layer="25" ratio="10"/>
+<attribute name="SPICEPREFIX" value="R" x="2.54" y="-24.13" size="1.778" layer="27" display="off"/>
+<attribute name="VALUE" x="0.4064" y="-26.4414" size="1.27" layer="27" ratio="10"/>
+</element>
+<element name="C1" library="rcl" library_urn="urn:adsk.eagle:library:334" package="C025-024X044" package3d_urn="urn:adsk.eagle:package:23630/1" value="0.1μ" x="1.27" y="-30.48" smashed="yes">
+<attribute name="NAME" x="-0.508" y="-29.083" size="1.27" layer="25" ratio="10"/>
+<attribute name="SPICEPREFIX" value="C" x="1.27" y="-30.48" size="1.778" layer="27" display="off"/>
+<attribute name="VALUE" x="-0.508" y="-33.147" size="1.27" layer="27" ratio="10"/>
+</element>
+<element name="C2" library="rcl" library_urn="urn:adsk.eagle:library:334" package="E5-10,5" package3d_urn="urn:adsk.eagle:package:23372/2" value="47μ" x="5.08" y="-38.1" smashed="yes">
+<attribute name="NAME" x="9.779" y="-35.3568" size="1.27" layer="25" ratio="10"/>
+<attribute name="SPICEPREFIX" value="C" x="5.08" y="-38.1" size="1.778" layer="27" display="off"/>
+<attribute name="VALUE" x="1.9558" y="-41.3258" size="1.27" layer="27" ratio="10"/>
+</element>
 </elements>
 <signals>
@@
 <contactref element="U$1" pad="P$29"/>
 </signal>
+<signal name="N$1">
+<contactref element="JP1" pad="2"/>
+<contactref element="Q1" pad="3"/>
+<contactref element="R1" pad="2"/>
+<wire x1="9.66" y1="-6.35" x2="22.86" y2="49.53" width="0" layer="19" extent="1-1"/>
+<wire x1="15.24" y1="26.67" x2="9.66" y2="-6.35" width="0" layer="19" extent="1-1"/>
+</signal>
+<signal name="N$2">
+<contactref element="Q1" pad="1"/>
+<contactref element="U$2" pad="2"/>
+<contactref element="R1" pad="1"/>
+<wire x1="5.08" y1="-6.35" x2="15.24" y2="34.29" width="0" layer="19" extent="1-1"/>
+<wire x1="12.7" y1="26.67" x2="5.08" y2="-6.35" width="0" layer="19" extent="1-1"/>
+</signal>
+<signal name="N$4">
+<contactref element="Q1" pad="2"/>
+<contactref element="R2" pad="2"/>
+<contactref element="R3" pad="2"/>
+<contactref element="IC1" pad="1"/>
+<contactref element="C1" pad="1"/>
+<wire x1="7.37" y1="-6.35" x2="24.13" y2="45.72" width="0" layer="19" extent="1-1"/>
+<wire x1="3.81" y1="-11.43" x2="7.37" y2="-6.35" width="0" layer="19" extent="1-1"/>
+<wire x1="3.81" y1="-17.78" x2="3.81" y2="-11.43" width="0" layer="19" extent="1-1"/>
+<wire x1="0" y1="-30.48" x2="3.81" y2="-17.78" width="0" layer="19" extent="1-1"/>
+</signal>
+<signal name="N$5">
+<contactref element="R2" pad="1"/>
+<contactref element="LED1" pad="A"/>
+<wire x1="1.27" y1="-11.43" x2="11.43" y2="15.24" width="0" layer="19" extent="1-1"/>
+</signal>
+<signal name="BATTERY">
+<contactref element="R3" pad="1"/>
+<contactref element="R4" pad="2"/>
+<wire x1="1.27" y1="-17.78" x2="3.81" y2="-24.13" width="0" layer="19" extent="1-1"/>
+</signal>
+<signal name="GND">
+<contactref element="JP1" pad="1"/>
+<contactref element="U$2" pad="1"/>
+<contactref element="LED1" pad="K"/>
+<contactref element="R4" pad="1"/>
+<contactref element="IC1" pad="2"/>
+<contactref element="C1" pad="2"/>
+<contactref element="C2" pad="-"/>
+<wire x1="21.83" y1="45.72" x2="25.4" y2="49.53" width="0" layer="19" extent="1-1"/>
+<wire x1="12.7" y1="34.29" x2="21.83" y2="45.72" width="0" layer="19" extent="1-1"/>
+<wire x1="13.97" y1="15.24" x2="12.7" y2="34.29" width="0" layer="19" extent="1-1"/>
+<wire x1="1.27" y1="-24.13" x2="13.97" y2="15.24" width="0" layer="19" extent="1-1"/>
+<wire x1="2.54" y1="-30.48" x2="1.27" y2="-24.13" width="0" layer="19" extent="1-1"/>
+<wire x1="7.62" y1="-38.1" x2="2.54" y2="-30.48" width="0" layer="19" extent="1-1"/>
+</signal>
+<signal name="+5V">
+<contactref element="IC1" pad="3"/>
+<contactref element="C2" pad="+"/>
+<wire x1="2.54" y1="-38.1" x2="19.53" y2="45.72" width="0" layer="19" extent="1-1"/>
+</signal>
 </signals>
 <mfgpreviewcolors>
@@
 </drawing>
 <compatibility>
+<note version="8.2" severity="warning">
+Since Version 8.2, EAGLE supports online libraries. The ids
+of those online libraries will not be understood (or retained)
+with this version.
+</note>
 <note version="8.3" severity="warning">
 Since Version 8.3, EAGLE supports URNs for individual library

Commit message: add:sensor
Parts:
- added LED2: (no value), led:LED3MM
- added Q2, Q3, Q4: RPR-220, RPR-220:RPR-220
- added R10, R6, R8: 19k, rcl:0204V
- added R5, R7, R9: 100, rcl:0204V
- added U1, U2: TA8428K(O,S), TA8428K(O_S):HSIP7-P-2.54_1
- R1: value 100k -> 10k
Connections:
- removed net 29_+3V3: U$1.P$29
- new net +3V3: Q2.1, Q2.4, Q3.1, Q3.4, Q4.1, Q4.4, U$1.P$29
- new net N$3: LED2.A, R1.1
- new net N$6: Q2.2, R5.2
- new net N$7: Q3.2, R7.2
- new net N$8: Q4.2, R9.2
- new net SEN_C: Q3.3, R8.2
- new net SEN_L: Q2.3, R6.2
- new net SEN_R: Q4.3, R10.2
- net GND: now also R10.1, R5.1, R6.1, R7.1, R8.1, R9.1
- net N$2: now also LED2.K; no longer R1.1

Commit message: schematic
Parts:
- added C3, C4: 100μ, rcl:E2,5-7
- added D1: (no value), diode:DO07
- added LED3, LED4, LED5: (no value), led:LED3MM
- added LS1: QMB-111GPN, QMB-111GPN:QMB111GPN
- added MOTOR_L, MOTOR_R: (no value), pinhead:1X02
- added Q5: 2SC1815GRTE2FT, 2SC1815GRTE2FT:2-5F1B
- added R11, R12, R13, R14: 100, rcl:0204V
- added S1, S2: (no value), switch-omron:B3F-10XX
- C2: value 47μ -> 100μ; device rcl:E5-10,5 -> rcl:E2,5-7
- moved C2 85.1 mm to (2.54, -123.2)
- moved U2 52.1 mm to (8.89, -149.9)
Connections:
- removed net 17_GND: U$1.P$17
- removed net 19_+5V: U$1.P$19
- removed net 4_GND: U$1.P$4
- new net BATT: C1.1, C3.+, C4.+, IC1.1, Q1.2, R2.2, R3.2, U1.7, U2.7
- new net LED_C: LED4.A, U$1.P$10
- new net LED_L: LED5.A, U$1.P$11
- new net LED_R: LED3.A, U$1.P$9
- new net MOTOR_L_1: U$1.P$12, U1.1
- new net MOTOR_L_2: U$1.P$13, U1.2
- new net MOTOR_R_1: U$1.P$1, U2.1
- new net MOTOR_R_2: U$1.P$2, U2.2
- new net N$10: LED3.K, R12.2
- new net N$11: LED4.K, R13.2
- new net N$12: LED5.K, R14.2
- new net N$9: D1.A, LS1.2, Q5.2
- new net OUTA_L: MOTOR_L.1, U1.3
- new net OUTA_R: MOTOR_R.1, U2.3
- new net SPEAKER: Q5.3, U$1.P$22
- new net SWITCH_L: S1.1, U$1.P$15
- new net SWITCH_R: S2.1, U$1.P$14
- new net _OUTA_L: MOTOR_L.2, U1.5
- new net _OUTA_R: MOTOR_R.2, U2.5
- net +3V3: now also R11.2
- net +5V: now also U$1.P$19
- net BATTERY: now also U$1.P$21
- net GND: now also C3.-, C4.-, Q5.1, R12.1, R13.1, R14.1, S1.4, S2.4, U$1.P$17, U$1.P$4, U1.4, U2.4
- net N$4: now also D1.C, LS1.1, R11.1; no longer C1.1, IC1.1, Q1.2, R2.2, R3.2
- net SEN_C: now also U$1.P$24
- net SEN_L: now also U$1.P$25
- net SEN_R: now also U$1.P$23

Commit message: comp
Parts:
- removed D1: (no value), diode:DO07
- removed LED1: (no value), led:LED3MM
- removed R2: 4.7k, rcl:0204V
- added D2: (no value), diode:D-2.5
- moved LED5 267.7 mm to (22.5, 64.0)
- moved LED4 260.3 mm to (42.5, 64.0)
- moved R14 256.6 mm to (23.0, 58.0), turned to 270 degrees
- moved LED3 248.8 mm to (62.5, 64.0)
- moved R12 248.2 mm to (61.0, 58.0), turned to 270 degrees
- moved R13 248.2 mm to (38.0, 58.0), turned to 270 degrees
- moved S2 222.9 mm to (21.6, 8.35)
- moved MOTOR_R 218.1 mm to (79.3, 58.1), turned to 90 degrees
- moved U2 217.7 mm to (74.2, 57.9), turned to 90 degrees
- moved S1 207.8 mm to (7.62, 8.35)
- moved C4 205.1 mm to (68.3, 55.9), turned to 270 degrees
- moved R11 203.6 mm to (7.11, 47.7), turned to 180 degrees
- moved Q5 189.3 mm to (6.35, 20.9)
- moved C3 187.2 mm to (16.7, 55.9), turned to 90 degrees
- moved LS1 185.4 mm to (7.62, 38.6), turned to 180 degrees
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Connections:
- removed net N$5: LED1.A, R2.1
- net BATT: no longer R2.2
- net GND: now also LED3.K, LED4.K, LED5.K; no longer LED1.K, R12.1, R13.1, R14.1
- net LED_C: now also R13.2; no longer LED4.A
- net LED_L: now also R14.2; no longer LED5.A
- net LED_R: now also R12.2; no longer LED3.A
- net N$10: now also LED3.A, R12.1; no longer LED3.K, R12.2
- net N$11: now also LED4.A, R13.1; no longer LED4.K, R13.2
- net N$12: now also LED5.A, R14.1; no longer LED5.K, R14.2
- net N$4: now also D2.C; no longer D1.C
- net N$9: now also D2.A; no longer D1.A
Routing:
- net GND: track 0.00 -> 278.8 mm, vias 0 -> 1
- net BATT: track 0.00 -> 126.2 mm
- net +3V3: track 0.00 -> 109.3 mm
- net SEN_R: track 0.00 -> 51.7 mm, vias 0 -> 2
- net SWITCH_L: track 0.00 -> 46.4 mm
- net SEN_L: track 0.00 -> 44.7 mm, vias 0 -> 2
- net SPEAKER: track 0.00 -> 43.4 mm
- net SEN_C: track 0.00 -> 43.1 mm, vias 0 -> 2
- net SWITCH_R: track 0.00 -> 41.6 mm
- net N$2: track 0.00 -> 29.8 mm
- net MOTOR_L_1: track 0.00 -> 29.3 mm
- net +5V: track 0.00 -> 26.4 mm
- net MOTOR_L_2: track 0.00 -> 25.7 mm
- net N$9: track 0.00 -> 25.3 mm
- net LED_R: track 0.00 -> 23.9 mm
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- added copper zone on layer 1, net GND
- added copper zone on layer 16, net GND
Other:
- board size 160 x 100 mm -> 85 x 75 mm
- board text added: "Mice linetracer"

Commit message: add:chassis
Parts:
- added D1: (no value), diode:D-2.5
- added R2: 10k, rcl:0204V
- R10, R6, R8: value 19k -> 10k
- R12, R13, R14: value 100 -> 220
- moved C1 1.27 mm to (62.2, 16.5)
Connections:
- net +5V: now also D1.A
- net BATT: now also D1.C
- net GND: now also R2.1
- net SPEAKER: now also R2.2
Routing:
- net GND: track 278.8 -> 743.6 mm, vias 1 -> 34
- net +5V: track 26.4 -> 30.7 mm
- net BATT: track 126.2 -> 130.5 mm
- net SPEAKER: track 43.4 -> 46.9 mm
- net SEN_L: track 44.7 -> 45.7 mm
Other:
- board text added: "+"
- board text added: "i"
- board text added: "o"
