File: eagle/project_l432/linetracer/linetracer.sch (EAGLE design)
At the start: 1 part

Commit message: add:pdf
Parts:
- added U$1: NUCLEO_L432KC, nucleo32.Ibr:NUCLEO_L432KC
Other:
- moved on the sheet: JP1
Changed lines of the file:
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@@
 <parts>
 <part name="JP1" library="pinhead" deviceset="PINHD-1X2" device="" package3d_urn="urn:adsk.eagle:package:22435/2"/>
+<part name="U$1" library="nucleo32.Ibr" deviceset="NUCLEO_L432KC" device=""/>
+<part name="FRAME1" library="frames" library_urn="urn:adsk.eagle:library:229" deviceset="A3L-LOC" device=""/>
 </parts>
 <sheets>
@@
 </plain>
 <instances>
-<instance part="JP1" gate="G$1" x="12.7" y="27.94" smashed="yes" rot="R180">
-<attribute name="NAME" x="19.05" y="22.225" size="1.778" layer="95" rot="R180"/>
-<attribute name="VALUE" x="19.05" y="33.02" size="1.778" layer="96" rot="R180"/>
+<instance part="JP1" gate="G$1" x="10.16" y="30.48" smashed="yes" rot="R180">
+<attribute name="NAME" x="16.51" y="24.765" size="1.778" layer="95" rot="R180"/>
+<attribute name="VALUE" x="16.51" y="35.56" size="1.778" layer="96" rot="R180"/>
+</instance>
+<instance part="U$1" gate="G$1" x="55.88" y="66.04" smashed="yes"/>
+<instance part="FRAME1" gate="G$1" x="2.54" y="0" smashed="yes">
+<attribute name="DRAWING_NAME" x="346.71" y="15.24" size="2.54" layer="94"/>
+<attribute name="LAST_DATE_TIME" x="346.71" y="10.16" size="2.286" layer="94"/>
+<attribute name="SHEET" x="360.045" y="5.08" size="2.54" layer="94"/>
 </instance>
 </instances>
@@
 </drawing>
 <compatibility>
+<note version="8.2" severity="warning">
+Since Version 8.2, EAGLE supports online libraries. The ids
+of those online libraries will not be understood (or retained)
+with this version.
+</note>
 <note version="8.3" severity="warning">
 Since Version 8.3, EAGLE supports URNs for individual library

Commit message: power
Parts:
- added C1: 0.1μ, rcl:C-EU025-024X044
- added C2: 47μ, rcl:CPOL-EUE5-10.5
- added IC1: TA4805S, TA4805S:TA4805S
- added LED1: (no value), led:LED3MM
- added Q1: IRFU5505PBF, IRFU5505PBF:IRFU5505PBF
- added R1, R3: 100k, rcl:R-EU_0204/2V
- added R2: 4.7k, rcl:R-EU_0204/2V
- added R4: 22k, rcl:R-EU_0204/2V
- added U$2: TOGGLE-SWITCH, toggle-switch:TOGGLE-SWITCH
Connections:
- new net +5V: C2.+, IC1.OUT
- new net BATTERY: R3.1, R4.2
- new net GND: C1.2, C2.-, IC1.GND, JP1.1, LED1.C, R4.1, U$2.1
- new net N$1: JP1.2, Q1.S, R1.2
- new net N$2: Q1.G, R1.1, U$2.2
- new net N$4: C1.1, IC1.IN, Q1.D, R2.2, R3.2
- new net N$5: LED1.A, R2.1
Other:
- moved on the sheet: JP1

Commit message: add:sensor
Parts:
- added LED2: (no value), led:LED3MM
- added Q2, Q3, Q4: RPR-220, RPR-220:RPR-220
- added R10, R6, R8: 19k, rcl:R-EU_0204/2V
- added R5, R7, R9: 100, rcl:R-EU_0204/2V
- added U1, U2: TA8428K(O,S), TA8428K(O_S):TA8428K(O,S)
- R1: value 100k -> 10k
Connections:
- new net +3V3: Q2.ANODE, Q2.COLLECTOR, Q3.ANODE, Q3.COLLECTOR, Q4.ANODE, Q4.COLLECTOR, U$1.29_+3V3
- new net N$3: LED2.A, R1.1
- new net N$6: Q2.CATHODE, R5.2
- new net N$7: Q3.CATHODE, R7.2
- new net N$8: Q4.CATHODE, R9.2
- new net SEN_C: Q3.EMITTER, R8.2
- new net SEN_L: Q2.EMITTER, R6.2
- new net SEN_R: Q4.EMITTER, R10.2
- net GND: now also R10.1, R5.1, R6.1, R7.1, R8.1, R9.1
- net N$2: now also LED2.C; no longer R1.1
Other:
- note added: "Power"
- note added: "SENSOR"
- moved on the sheet: U$2

Commit message: schematic
Parts:
- added C3, C4: 100μ, rcl:CPOL-EUE2.5-7
- added D1: (no value), diode:DIODE-DO07
- added LED3, LED4, LED5: (no value), led:LED3MM
- added LS1: QMB-111GPN, QMB-111GPN:QMB-111GPN
- added MOTOR_L, MOTOR_R: (no value), pinhead:PINHD-1X2
- added Q5: 2SC1815GRTE2FT, 2SC1815GRTE2FT:2SC1815GRTE2FT
- added R11, R12, R13, R14: 100, rcl:R-EU_0204/2V
- added S1, S2: (no value), switch-omron:10-XX
- C2: value 47μ -> 100μ; device rcl:CPOL-EUE5-10.5 -> rcl:CPOL-EUE2.5-7
Connections:
- new net BATT: C1.1, C3.+, C4.+, IC1.IN, Q1.D, R2.2, R3.2, U1.VCC, U2.VCC
- new net LED_C: LED4.A, U$1.10_PC14
- new net LED_L: LED5.A, U$1.11_PC15
- new net LED_R: LED3.A, U$1.9_PB1
- new net MOTOR_L_1: U$1.12_PA8, U1.IN1
- new net MOTOR_L_2: U$1.13_PA11, U1.IN2
- new net MOTOR_R_1: U$1.1_PA9, U2.IN1
- new net MOTOR_R_2: U$1.2_PA10, U2.IN2
- new net N$10: LED3.C, R12.2
- new net N$11: LED4.C, R13.2
- new net N$12: LED5.C, R14.2
- new net N$9: D1.A, LS1.2, Q5.C
- new net OUTA_L: MOTOR_L.1, U1.OUTA
- new net OUTA_R: MOTOR_R.1, U2.OUTA
- new net SPEAKER: Q5.B, U$1.22_PA6
- new net SWITCH_L: S1.S, U$1.15_PB4
- new net SWITCH_R: S2.S, U$1.14_PB5
- new net _OUTA_L: MOTOR_L.2, U1.OUT_!A
- new net _OUTA_R: MOTOR_R.2, U2.OUT_!A
- net +3V3: now also R11.2
- net +5V: now also U$1.19_+5V
- net BATTERY: now also U$1.21_PA7
- net GND: now also C3.-, C4.-, Q5.E, R12.1, R13.1, R14.1, S1.P1, S2.P1, U$1.17_GND, U$1.4_GND, U1.GND, U2.GND
- net N$4: now also D1.C, LS1.1, R11.1; no longer C1.1, IC1.IN, Q1.D, R2.2, R3.2
- net SEN_C: now also U$1.24_PA4
- net SEN_L: now also U$1.25_PA3
- net SEN_R: now also U$1.23_PA5
Other:
- note added: "CPU"
- note added: "MOTOR"
- note added: "UI"
- moved on the sheet: C1, C2, IC1, JP1, LED1, LED2, Q1, R1, R2, R3, R4, U$2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

Commit message: comp
Parts:
- removed D1: (no value), diode:DIODE-DO07
- removed LED1: (no value), led:LED3MM
- removed R2: 4.7k, rcl:R-EU_0204/2V
- added D2: (no value), diode:DIODE-D-2.5
Connections:
- removed net N$5: LED1.A, R2.1
- net BATT: no longer R2.2
- net GND: now also LED3.C, LED4.C, LED5.C; no longer LED1.C, R12.1, R13.1, R14.1
- net LED_C: now also R13.2; no longer LED4.A
- net LED_L: now also R14.2; no longer LED5.A
- net LED_R: now also R12.2; no longer LED3.A
- net N$10: now also LED3.A, R12.1; no longer LED3.C, R12.2
- net N$11: now also LED4.A, R13.1; no longer LED4.C, R13.2
- net N$12: now also LED5.A, R14.1; no longer LED5.C, R14.2
- net N$4: now also D2.C; no longer D1.C
- net N$9: now also D2.A; no longer D1.A
Other:
- moved on the sheet: C3, LED3, LED4, LED5, MOTOR_L, Q2, Q3, Q4, R10, R12, R13, R14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

Commit message: add:chassis
Parts:
- added D1: (no value), diode:DIODE-D-2.5
- added R2: 10k, rcl:R-EU_0204/2V
- R10, R6, R8: value 19k -> 10k
- R12, R13, R14: value 100 -> 220
Connections:
- net +5V: now also D1.A
- net BATT: now also D1.C
- net GND: now also R2.1
- net SPEAKER: now also R2.2
Changed lines of the file:
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@@
 <part name="R5" library="rcl" library_urn="urn:adsk.eagle:library:334" deviceset="R-EU_" device="0204/2V" package3d_urn="urn:adsk.eagle:package:23495/1" value="100"/>
 <part name="GND2" library="supply1" library_urn="urn:adsk.eagle:library:371" deviceset="GND" device=""/>
-<part name="R6" library="rcl" library_urn="urn:adsk.eagle:library:334" deviceset="R-EU_" device="0204/2V" package3d_urn="urn:adsk.eagle:package:23495/1" value="19k"/>
+<part name="R6" library="rcl" library_urn="urn:adsk.eagle:library:334" deviceset="R-EU_" device="0204/2V" package3d_urn="urn:adsk.eagle:package:23495/1" value="10k"/>
 <part name="GND3" library="supply1" library_urn="urn:adsk.eagle:library:371" deviceset="GND" device=""/>
 <part name="Q3" library="RPR-220" deviceset="RPR-220" device=""/>
@@
 <part name="R7" library="rcl" library_urn="urn:adsk.eagle:library:334" deviceset="R-EU_" device="0204/2V" package3d_urn="urn:adsk.eagle:package:23495/1" value="100"/>
 <part name="GND4" library="supply1" library_urn="urn:adsk.eagle:library:371" deviceset="GND" device=""/>
-<part name="R8" library="rcl" library_urn="urn:adsk.eagle:library:334" deviceset="R-EU_" device="0204/2V" package3d_urn="urn:adsk.eagle:package:23495/1" value="19k"/>
+<part name="R8" library="rcl" library_urn="urn:adsk.eagle:library:334" deviceset="R-EU_" device="0204/2V" package3d_urn="urn:adsk.eagle:package:23495/1" value="10k"/>
 <part name="GND5" library="supply1" library_urn="urn:adsk.eagle:library:371" deviceset="GND" device=""/>
 <part name="Q4" library="RPR-220" deviceset="RPR-220" device=""/>
@@
 <part name="R9" library="rcl" library_urn="urn:adsk.eagle:library:334" deviceset="R-EU_" device="0204/2V" package3d_urn="urn:adsk.eagle:package:23495/1" value="100"/>
 <part name="GND6" library="supply1" library_urn="urn:adsk.eagle:library:371" deviceset="GND" device=""/>
-<part name="R10" library="rcl" library_urn="urn:adsk.eagle:library:334" deviceset="R-EU_" device="0204/2V" package3d_urn="urn:adsk.eagle:package:23495/1" value="19k"/>
+<part name="R10" library="rcl" library_urn="urn:adsk.eagle:library:334" deviceset="R-EU_" device="0204/2V" package3d_urn="urn:adsk.eagle:package:23495/1" value="10k"/>
 <part name="GND7" library="supply1" library_urn="urn:adsk.eagle:library:371" deviceset="GND" device=""/>
 <part name="+3V5" library="supply1" library_urn="urn:adsk.eagle:library:371" deviceset="+3V3" device=""/>
@@
 <part name="LED4" library="led" library_urn="urn:adsk.eagle:library:259" deviceset="LED" device="3MM" package3d_urn="urn:adsk.eagle:package:15797/1"/>
 <part name="LED5" library="led" library_urn="urn:adsk.eagle:library:259" deviceset="LED" device="3MM" package3d_urn="urn:adsk.eagle:package:15797/1"/>
-<part name="R12" library="rcl" library_urn="urn:adsk.eagle:library:334" deviceset="R-EU_" device="0204/2V" package3d_urn="urn:adsk.eagle:package:23495/1" value="100"/>
-<part name="R13" library="rcl" library_urn="urn:adsk.eagle:library:334" deviceset="R-EU_" device="0204/2V" package3d_urn="urn:adsk.eagle:package:23495/1" value="100"/>
-<part name="R14" library="rcl" library_urn="urn:adsk.eagle:library:334" deviceset="R-EU_" device="0204/2V" package3d_urn="urn:adsk.eagle:package:23495/1" value="100"/>
+<part name="R12" library="rcl" library_urn="urn:adsk.eagle:library:334" deviceset="R-EU_" device="0204/2V" package3d_urn="urn:adsk.eagle:package:23495/1" value="220"/>
+<part name="R13" library="rcl" library_urn="urn:adsk.eagle:library:334" deviceset="R-EU_" device="0204/2V" package3d_urn="urn:adsk.eagle:package:23495/1" value="220"/>
+<part name="R14" library="rcl" library_urn="urn:adsk.eagle:library:334" deviceset="R-EU_" device="0204/2V" package3d_urn="urn:adsk.eagle:package:23495/1" value="220"/>
+<part name="R2" library="rcl" library_urn="urn:adsk.eagle:library:334" deviceset="R-EU_" device="0204/2V" package3d_urn="urn:adsk.eagle:package:23495/1" value="10k"/>
+<part name="D1" library="diode" library_urn="urn:adsk.eagle:library:210" deviceset="DIODE-" device="D-2.5" package3d_urn="urn:adsk.eagle:package:43419/1"/>
 </parts>
 <sheets>
@@
 <attribute name="VALUE" x="51.562" y="189.23" size="1.778" layer="96" rot="R90"/>
 </instance>
+<instance part="R2" gate="G$1" x="53.34" y="106.68" smashed="yes" rot="R180">
+<attribute name="NAME" x="57.15" y="105.1814" size="1.778" layer="95" rot="R180"/>
+<attribute name="VALUE" x="57.15" y="109.982" size="1.778" layer="96" rot="R180"/>
+</instance>
+<instance part="D1" gate="G$1" x="355.6" y="147.32" smashed="yes" rot="R180">
+<attribute name="NAME" x="353.06" y="146.8374" size="1.778" layer="95" rot="R180"/>
+<attribute name="VALUE" x="353.06" y="149.6314" size="1.778" layer="96" rot="R180"/>
+</instance>
 </instances>
 <busses>
@@
 <wire x1="330.2" y1="119.38" x2="330.2" y2="127" width="0.1524" layer="91"/>
 <pinref part="VDD1" gate="G$1" pin="VDD"/>
+<wire x1="347.98" y1="119.38" x2="347.98" y2="147.32" width="0.1524" layer="91"/>
+<pinref part="D1" gate="G$1" pin="C"/>
+<wire x1="347.98" y1="147.32" x2="353.06" y2="147.32" width="0.1524" layer="91"/>
 </segment>
 <segment>
@@
 <wire x1="60.96" y1="106.68" x2="60.96" y2="104.14" width="0.1524" layer="91"/>
 <pinref part="GND12" gate="1" pin="GND"/>
+<pinref part="R2" gate="G$1" pin="1"/>
+<wire x1="58.42" y1="106.68" x2="60.96" y2="106.68" width="0.1524" layer="91"/>
+<junction x="60.96" y="106.68"/>
 </segment>
 <segment>
@@
 <pinref part="IC1" gate="G$1" pin="OUT"/>
 <wire x1="358.14" y1="119.38" x2="360.68" y2="119.38" width="0.1524" layer="91"/>
-<wire x1="360.68" y1="119.38" x2="365.76" y2="119.38" width="0.1524" layer="91"/>
+<wire x1="360.68" y1="119.38" x2="363.22" y2="119.38" width="0.1524" layer="91"/>
+<wire x1="363.22" y1="119.38" x2="365.76" y2="119.38" width="0.1524" layer="91"/>
 <wire x1="365.76" y1="119.38" x2="365.76" y2="121.92" width="0.1524" layer="91"/>
 <pinref part="P+1" gate="1" pin="+5V"/>
 <pinref part="C2" gate="G$1" pin="+"/>
 <junction x="360.68" y="119.38"/>
+<pinref part="D1" gate="G$1" pin="A"/>
+<wire x1="358.14" y1="147.32" x2="363.22" y2="147.32" width="0.1524" layer="91"/>
+<wire x1="363.22" y1="147.32" x2="363.22" y2="119.38" width="0.1524" layer="91"/>
+<junction x="363.22" y="119.38"/>
 </segment>
 </net>
@@
 <segment>
 <pinref part="Q5" gate="G$1" pin="B"/>
-<wire x1="50.8" y1="114.3" x2="43.18" y2="114.3" width="0.1524" layer="91"/>
+<wire x1="50.8" y1="114.3" x2="45.72" y2="114.3" width="0.1524" layer="91"/>
 <label x="43.18" y="114.3" size="1.4224" layer="95" rot="R180" xref="yes"/>
-</segment>
-</net>
+<pinref part="R2" gate="G$1" pin="2"/>
+<wire x1="45.72" y1="114.3" x2="43.18" y2="114.3" width="0.1524" layer="91"/>
+<wire x1="48.26" y1="106.68" x2="45.72" y2="106.68" width="0.1524" layer="91"/>
+<wire x1="45.72" y1="106.68" x2="45.72" y2="114.3" width="0.1524" layer="91"/>
+<junction x="45.72" y="114.3"/>
+</segment>
+</net>
